File: pcb/splitflap-berlin.kicad_pcb (KiCad board)
At the start: 2 copper layers, 100 x 100 mm, 64 parts, among them J1 Screw_Terminal_01x02, J2 Conn_02x05_Odd_Even, J3 Conn_02x05_Odd_Even, J4 Conn_02x05_Odd_Even, Q1 BT136-600, Q2 BT136-600, Q3 BT136-600, T1 Transformer_1P_2S, T2 Transformer_1P_1S, U1 MOC3041M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

Commit message: opened with newer kicad-version
Other:
- net class 230VAC removed
- net class 48VAC removed
- net class Default removed
